Commit message: modified urdf files

File: wonik_real/robot_model/urdf/wonik_robot_xacros/body.xacro (robot description, xacro)
@@ -22,5 +22,5 @@
         <origin xyz="0. 0. 0" rpy="-1.571 0 1.571" />
         <geometry>
-            <mesh filename="package://wonik_robot/robot_model/meshes/wonik_robot/BODY.dae" scale="0.001 0.001 0.001"/>
+            <mesh filename="package://wonik_real/robot_model/meshes/wonik_robot/BODY.dae" scale="0.001 0.001 0.001"/>
         </geometry>
       </visual>
@@ -29,5 +29,5 @@
         <geometry>
           <!--<box size="0.68 0.41 0.25"/> -->
-          <mesh filename="package://wonik_robot/robot_model/meshes/wonik_robot/BODY.dae" scale="0.001 0.001 0.001"/>
+          <mesh filename="package://wonik_real/robot_model/meshes/wonik_robot/BODY.dae" scale="0.001 0.001 0.001"/>
         </geometry>
       </collision>

File: wonik_real/robot_model/urdf/wonik_robot_xacros/cabinet.xacro (robot description, xacro)
@@ -19,5 +19,5 @@
         <origin xyz="0 0 0" rpy="0 0 -1.5708" />
         <geometry>
-            <mesh filename="package://neo_mpo_500/robot_model/meshes/MPO_500/cabin.dae" scale="0.001 0.001 0.001"/>
+            <mesh filename="package://wonik_real/robot_model/meshes/wonik_robot/cabin.dae" scale="0.001 0.001 0.001"/>
         </geometry>
       </visual>
@@ -25,5 +25,5 @@
         <origin xyz="0. 0. 0" rpy="0 0 0" />
         <geometry>
-            <mesh filename="package://neo_mpo_500/robot_model/meshes/MPO_500/cabin.dae" scale="0.001 0.001 0.001"/>
+            <mesh filename="package://wonik_real/robot_model/meshes/wonik_robot/cabin.dae" scale="0.001 0.001 0.001"/>
         </geometry>
       </collision>

File: wonik_real/robot_model/urdf/wonik_robot_xacros/omni_wheel.xacro (robot description, xacro)
@@ -20,5 +20,5 @@
      <origin xyz="0 0 0" rpy="0 0 0"/>
      <geometry>
-        <mesh filename="package://wonik_robot/robot_model/meshes/wonik_robot/MPO-500-WHEEL.dae" scale="0.001 0.001 0.001"/>
+        <mesh filename="package://wonik_real/robot_model/meshes/wonik_robot/WHEEL.dae" scale="0.001 0.001 0.001"/>
      </geometry>
     </visual>
@@ -26,5 +26,5 @@
      <origin xyz="0 0 0" rpy="0 0 0" />
      <geometry>
-        <mesh filename="package://wonik_robot/robot_model/meshes/wonik_robot/MPO-500-WHEEL.dae" scale="0.001 0.001 0.001"/>
+        <mesh filename="package://wonik_real/robot_model/meshes/wonik_robot/WHEEL.dae" scale="0.001 0.001 0.001"/>
      </geometry>
     </collision>

File: wonik_real/robot_model/urdf/wonik_robot_xacros/sick_S561.xacro (robot description, xacro)
@@ -17,5 +17,5 @@
         <origin xyz="0 0 -0.12" rpy="-1.57 0 3.14" />
         <geometry>
-        <mesh filename="package://wonik_robot/robot_model/meshes/wonik_robot/SICK-S561.dae" scale="0.001 0.001 0.001" />
+        <mesh filename="package://wonik_real/robot_model/meshes/wonik_robot/SICK-S561.dae" scale="0.001 0.001 0.001" />
         </geometry>
       </visual>
@@ -23,5 +23,5 @@
         <origin xyz="0 0 -0.12" rpy="-1.57 0 3.14" />
         <geometry>
-        <mesh filename="package://wonik_robot/robot_model/meshes/wonik_robot/SICK-S561.dae" scale="0.001 0.001 0.001" />
+        <mesh filename="package://wonik_real/robot_model/meshes/wonik_robot/SICK-S561.dae" scale="0.001 0.001 0.001" />
         </geometry>
       </collision>

File: wonik_real/robot_model/urdf/wonik_robot_xacros/sick_laser.xacro (robot description, xacro)
@@ -18,5 +18,5 @@
       <origin xyz="0 0 -0.12" rpy="-1.57 0 3.14" />
         <geometry>
-        <mesh filename="package://wonik_robot/robot_model/meshes/wonik_robot/SICK-S300.dae" scale="0.001 0.001 0.001" />
+        <mesh filename="package://wonik_real/robot_model/meshes/wonik_robot/SICK-S300.dae" scale="0.001 0.001 0.001" />
         </geometry>
       </visual>
@@ -24,5 +24,5 @@
         <origin xyz="0 0 0" rpy="-1.57 0 3.14" />
         <geometry>
-        <mesh filename="package://wonik_robot/robot_model/meshes/wonik_robot/SICK-S300.dae" scale="0.001 0.001 0.001" />
+        <mesh filename="package://wonik_real/robot_model/meshes/wonik_robot/SICK-S300.dae" scale="0.001 0.001 0.001" />
         </geometry>
       </collision>

File: wonik_real/robot_model/wonik_robot.urdf.xacro (robot description, xacro)
@@ -8,5 +8,5 @@
   <xacro:include filename="$(find wonik_real)/robot_model/urdf/wonik_robot_xacros/sick_S561.xacro" />
   <!-- USS and IMU - Comment/Uncomment if required  -->
-  <!--<xacro:include filename="$(find wonik_real)/robot_model/urdf/wonik_robot_xacros/imu.xacro" /> -->
+  <xacro:include filename="$(find wonik_real)/robot_model/urdf/wonik_robot_xacros/imu.xacro" />
   <!-- CABINET -->
   <xacro:include filename="$(find wonik_real)/robot_model/urdf/wonik_robot_xacros/cabinet.xacro" />
@@ -39,7 +39,7 @@
      <!--+++++++++++++++++++ IMU ++++++++++++++++++++++++-->
  <!-- Comment or uncomment based on your requirement -->
-<!--   <xacro:imu name="imu_1" parent="base_link">
+  <xacro:imu name="imu_1" parent="base_link">
     <origin xyz="0.100 0 0.300" rpy="0 0 3.14" />
-  </xacro:imu> -->
+  </xacro:imu>
     <!--Camera  -->
 <!-- <xacro:camera name="camera" parent="base_link">
@@ -47,7 +47,6 @@
   </xacro:camera> -->
   <!--cabinet-->
-<!--   <xacro:wonik_robot_cabinet name="cabinet" parent="base_link">
+  <!-- <xacro:cabinet name="cabinet" parent="base_link">
   	<origin xyz="0.072 0 0.386" rpy="0 0 0" />
-  </xacro:wonik_robot_cabinet>
- -->
+  </xacro:cabinet> -->
 </robot>
