Commit message: fix bug for override

File: wonik_real/robot_model/urdf/wonik_robot_xacros/sick_S561.xacro (robot description, xacro)
@@ -15,5 +15,5 @@
       </inertial>
       <visual>
-        <origin xyz="0 0 -0.12" rpy="-1.57 0 3.14" />
+        <origin xyz="0 0 0" rpy="-1.57 0 3.14" />
         <geometry>
         <mesh filename="package://wonik_real/robot_model/meshes/wonik_robot/SICK-S561.dae" scale="0.001 0.001 0.001" />
@@ -21,5 +21,5 @@
       </visual>
       <collision>
-        <origin xyz="0 0 -0.12" rpy="-1.57 0 3.14" />
+        <origin xyz="0 0 0" rpy="-1.57 0 3.14" />
         <geometry>
         <mesh filename="package://wonik_real/robot_model/meshes/wonik_robot/SICK-S561.dae" scale="0.001 0.001 0.001" />

File: wonik_real/robot_model/wonik_robot.urdf.xacro (robot description, xacro)
@@ -32,8 +32,8 @@
   <!-- Sensors -->
   <xacro:sick_laser_v0 name="lidar_1" parent="base_link" ros_topic="lidar_1/scan">
-    <origin xyz="0.463193 0.310743 0.18904" rpy="0 0 0" />
+    <origin xyz="0.463193 0.320743 0.18904" rpy="3.14 0 0.785" />
   </xacro:sick_laser_v0>
   <xacro:sick_laser_v0 name="lidar_2" parent="base_link" ros_topic="lidar_2/scan">
-    <origin xyz="-0.463193 -0.310743 0.18904" rpy="3.14 0 3.14" />
+    <origin xyz="-0.463193 -0.320743 0.18904" rpy="3.14 0 3.925" />
   </xacro:sick_laser_v0>
      <!--+++++++++++++++++++ IMU ++++++++++++++++++++++++-->
