Commit message: update driver for motors

File: wonik_simulation/robots/wonik_robot.urdf.xacro (robot description, xacro)
@@ -12,8 +12,5 @@
   <xacro:include filename="$(find wonik_simulation)/robots/xacros/micro_scan.xacro" />
   <!--Ultrasonics, cameras and IMU's  -->
-  <!-->
-  <xacro:include filename="$(find wonik_simulation)/robots/wonik_robot/xacros/imu.xacro" />
-  <xacro:include filename="$(find wonik_simulation)/robots/wonik_robot/xacros/ultrasonic.xacro" />
-  <-->
+  <xacro:include filename="$(find wonik_simulation)/robots/xacros/imu.xacro" />
   <!-- <xacro:include filename="$(find wonik_simulation)/robots/wonik_robot/xacros/camera.xacro" />  -->
   <link name="base_link" />
@@ -44,77 +41,7 @@
   <!--+++++++++++++++++++ IMU ++++++++++++++++++++++++-->
   <!-- Comment or uncomment based on your requirement -->
-  <!-->
   <xacro:imu name="imu" parent="base_link">
     <origin xyz="0.100 0 0.300" rpy="0 0 3.14" />
   </xacro:imu>
-  <-->
-  <!--+++++++++++++++++++ Ultra Sonic ++++++++++++++++++++++++-->
-  <!-- Comment or uncomment based on your requirement -->
-  <!-- SENSOR 1 -->
-  <!-->
-  <xacro:us_sensor name="us_1" parent="base_link">
-    <origin xyz="0.100 0 0.500" rpy="0 3.14 3.14" />
-  </xacro:us_sensor>
-  <-->
-  <!-- SENSOR 2 -->
-  <!-- xacro:us_sensor name="us_2" parent="base_link">
-    <origin xyz="0.110 0 0.300" rpy="0 3.14 3.14" />
-  </xacro:us_sensor-->
-  <!-- SENSOR 3 -->
-  <!-- xacro:us_sensor name="us_3" parent="base_link">
-    <origin xyz="0.120 0 0.300" rpy="0 3.14 3.14" />
-  </xacro:us_sensor-->
-  <!-- SENSOR 4 -->
-  <!-- xacro:us_sensor name="us_4" parent="base_link">
-    <origin xyz="0.130 0 0.300" rpy="0 3.14 3.14" />
-  </xacro:us_sensor-->
-  <!-- SENSOR 5 -->
-  <!-- xacro:us_sensor name="us_5" parent="base_link">
-    <origin xyz="0.140 0 0.300" rpy="0 3.14 3.14" />
-  </xacro:us_sensor-->
-  <!-- SENSOR 6 -->
-  <!-- xacro:us_sensor name="us_6" parent="base_link">
-    <origin xyz="0.150 0 0.300" rpy="0 3.14 3.14" />
-  </xacro:us_sensor-->
-  <!-- SENSOR 7 -->
-  <!-- xacro:us_sensor name="us_7" parent="base_link">
-    <origin xyz="0.160 0 0.300" rpy="0 3.14 3.14" />
-  </xacro:us_sensor-->
-  <!-- SENSOR 8 -->
-  <!-- xacro:us_sensor name="us_8" parent="base_link">
-    <origin xyz="0.170 0 0.300" rpy="0 3.14 3.14" />
-  </xacro:us_sensor-->
-  <!-- SENSOR 9 -->
-  <!-- xacro:us_sensor name="us_9" parent="base_link">
-    <origin xyz="0.180 0 0.300" rpy="0 3.14 3.14" />
-  </xacro:us_sensor-->
-  <!-- SENSOR 10 -->
-  <!-- xacro:us_sensor name="us_10" parent="base_link">
-    <origin xyz="0.100 0 0.300" rpy="0 3.14 3.14" />
-  </xacro:us_sensor-->
-  <!-- SENSOR 11 -->
-  <!-- xacro:us_sensor name="us_11" parent="base_link">
-    <origin xyz="0.100 0 0.300" rpy="0 3.14 3.14" />
-  </xacro:us_sensor-->
-  <!-- SENSOR 12 -->
-  <!-- xacro:us_sensor name="us_12" parent="base_link">
-    <origin xyz="0.190 0 0.300" rpy="0 3.14 3.14" />
-  </xacro:us_sensor-->
-  <!-- SENSOR 13 -->
-  <!-- xacro:us_sensor name="us_13" parent="base_link">
-    <origin xyz="0.200 0 0.300" rpy="0 3.14 3.14" />
-  </xacro:us_sensor-->
-  <!-- SENSOR 14 -->
-  <!-- xacro:us_sensor name="us_14" parent="base_link">
-    <origin xyz="0.210 0 0.300" rpy="0 3.14 3.14" />
-  </xacro:us_sensor-->
-  <!-- SENSOR 15 -->
-  <!-- xacro:us_sensor name="us_15" parent="base_link">
-    <origin xyz="0.220 0 0.300" rpy="0 3.14 3.14" />
-  </xacro:us_sensor-->
-  <!-- SENSOR 16 -->
-  <!-- xacro:us_sensor name="us_16" parent="base_link">
-    <origin xyz="0.230 0 0.300" rpy="0 3.14 3.14" />
-  </xacro:us_sensor-->
   <!--Camera  -->
 <!-- <xacro:camera name="camera" parent="base_link">

File: wonik_simulation/robots/xacros/imu.xacro (robot description, xacro)
@@ -1,4 +1,4 @@
 <?xml version="1.0"?>
-<robot xmlns:xacro="http://www.ros.org/wiki/xacro" name="mp_400">
+<robot xmlns:xacro="http://www.ros.org/wiki/xacro" name="wonik_robot">
   <xacro:macro name="imu" params="name parent *origin">
     <joint name="${name}_joint" type="fixed">

File: wonik_simulation/robots/xacros/wonik_robot_gazebo.xacro (robot description, xacro)
@@ -110,22 +110,16 @@
    </gazebo>
   <!-- IMU sensor -->
-  <gazebo reference="imu_link">
-    <gravity>true</gravity>
-    <sensor name="imu_sensor" type="imu">
-      <always_on>true</always_on>
-      <update_rate>100</update_rate>
-      <visualize>true</visualize>
-      <topic>__default_topic__</topic>
-      <plugin filename="libgazebo_ros_imu_sensor.so" name="imu_plugin">
-        <topicName>imu</topicName>
-        <bodyName>imu_link</bodyName>
-        <updateRateHZ>10.0</updateRateHZ>
-        <gaussianNoise>0.0</gaussianNoise>
-        <xyzOffset>0 0 0</xyzOffset>
-        <rpyOffset>0 0 0</rpyOffset>
-        <frameName>imu_link</frameName>
-      </plugin>
-      <pose>0 0 0 0 0 0</pose>
-    </sensor>
+  <gazebo>
+    <plugin name="imu_controller" filename="libhector_gazebo_ros_imu.so">
+      <updateRate>500.0</updateRate>
+      <bodyName>imu_link</bodyName>
+      <topicName>imu/data</topicName>
+      <accelDrift>0.005 0.005 0.005</accelDrift>
+      <accelGaussianNoise>0.005 0.005 0.005</accelGaussianNoise>
+      <rateDrift>0.005 0.005 0.005 </rateDrift>
+      <rateGaussianNoise>0.005 0.005 0.005 </rateGaussianNoise>
+      <headingDrift>0.005</headingDrift>
+      <headingGaussianNoise>0.005</headingGaussianNoise>
+    </plugin>
   </gazebo>
   <!-- Ultrasonic sensors -->
