Commit message: update sf factor

File: wonik_real/robot_model/wonik_robot.urdf.xacro (robot description, xacro)
@@ -18,22 +18,22 @@
   </xacro:wonik_robot_base>
   <!-- Wheel Macro -->
-  <xacro:omni_wheel_250 name="wonik_robot_wheel_front_left" parent="base_footprint">
+  <xacro:omni_wheel_250 name="wheel_front_left" parent="base_footprint">
   	<origin xyz="0.25 0.28 0.13" rpy="0 0 0" />
   </xacro:omni_wheel_250>
-  <xacro:omni_wheel_250 name="wonik_robot_wheel_front_right" parent="base_footprint">
+  <xacro:omni_wheel_250 name="wheel_front_right" parent="base_footprint">
   	<origin xyz="0.25 -0.28 0.13" rpy="0 0 3.14" />
   </xacro:omni_wheel_250>
-  <xacro:omni_wheel_250 name="wonik_robot_wheel_back_left" parent="base_footprint">
+  <xacro:omni_wheel_250 name="wheel_rear_left" parent="base_footprint">
   	<origin xyz="-0.25 0.28 0.13" rpy="0 0 0" />
   </xacro:omni_wheel_250>
-  <xacro:omni_wheel_250 name="wonik_robot_wheel_back_right" parent="base_footprint">
+  <xacro:omni_wheel_250 name="wheel_rear_right" parent="base_footprint">
   	<origin xyz="-0.25 -0.28 0.13" rpy="0 0 3.14" />
   </xacro:omni_wheel_250>
   <!-- Sensors -->
   <xacro:sick_laser_v0 name="lidar_1" parent="base_link" ros_topic="lidar_1/scan">
-    <origin xyz="0.442 0 0.372" rpy="0 0 0" />
+    <origin xyz="0.463193 0.310743 0.18904" rpy="0 0 0" />
   </xacro:sick_laser_v0>
   <xacro:sick_laser_v0 name="lidar_2" parent="base_link" ros_topic="lidar_2/scan">
-    <origin xyz="-0.442 0 0.372" rpy="0 0 3.14" />
+    <origin xyz="-0.463193 -0.310743 0.18904" rpy="3.14 0 3.14" />
   </xacro:sick_laser_v0>
      <!--+++++++++++++++++++ IMU ++++++++++++++++++++++++-->

Commit message: fix imu bug

File: wonik_real/robot_model/wonik_robot.urdf.xacro (robot description, xacro)
@@ -40,5 +40,5 @@
  <!-- Comment or uncomment based on your requirement -->
   <xacro:imu name="imu" parent="base_link">
-    <origin xyz="0.100 0 0.300" rpy="0 0 3.14" />
+    <origin xyz="0.100 0 0.300" rpy="0 0 0" />
   </xacro:imu>
     <!--Camera  -->

Commit message: update threads

File: wonik_real/robot_model/wonik_robot.urdf.xacro (robot description, xacro)
@@ -7,4 +7,5 @@
   <!-- SENSORS -->
   <xacro:include filename="$(find wonik_real)/robot_model/urdf/wonik_robot_xacros/sick_S561.xacro" />
+  <xacro:include filename="$(find wonik_real)/robot_model/urdf/wonik_robot_xacros/d435.xacro" />
   <!-- USS and IMU - Comment/Uncomment if required  -->
   <xacro:include filename="$(find wonik_real)/robot_model/urdf/wonik_robot_xacros/imu.xacro" />
@@ -37,4 +38,10 @@
     <origin xyz="-0.463193 -0.320743 0.18904" rpy="3.14 0 3.925" />
   </xacro:sick_laser_v0>
+  <xacro:camera_v0 name="cam_1" parent="base_link" ros_topic="cam_1/scan">
+    <origin xyz="0.463193 0.038242 0.53424" rpy="1.5707 -0.174533 0.3054326" />
+  </xacro:camera_v0>
+  <xacro:camera_v0 name="cam_2" parent="base_link" ros_topic="cam_2/scan">
+    <origin xyz="0.463193 -0.038242 0.53424" rpy="1.5707 -0.174533 -0.3054326" />
+  </xacro:camera_v0>
      <!--+++++++++++++++++++ IMU ++++++++++++++++++++++++-->
  <!-- Comment or uncomment based on your requirement -->
